File: BulkyModem Module/c64_userport.sch (KiCad schematic (older format))
At the start: 1 part, among them J4 C64_User_Port

Commit message: C64 UserPort adapter sketched out (preliminary layout)
Parts:
- removed J4: C64_User_Port, symbol c64_user_port:C64_User_Port
- added J5: C64_Modem_IDC, BulkyModem:C64_Adapter_IDC, symbol c64_adapter_idc:C64_Modem_OUT
Connections:
- net labels added: +5V, GND
- wire segments 0 -> 16
- no-connect marks 24 -> 0
Changed lines of the file:
@@
 encoding utf-8
 Sheet 4 5
-Title ""
+Title "BulkyModem Module (C64 UserPort)"
 Date ""
-Rev ""
+Rev "A"
 Comp ""
 Comment1 ""
@@
 Comment4 ""
 $EndDescr
+Text HLabel 5375 3800 0    50   Input ~ 0
+C64_TX
+Text HLabel 5375 4000 0    50   Input ~ 0
+C64_RTS
+Text HLabel 5375 3900 0    50   Output ~ 0
+C64_RX
+Text HLabel 5375 4100 0    50   Output ~ 0
+C64_CTS
 $Comp
-L c64_user_port:C64_User_Port J4
-U 1 1 63AED972
-P 5075 3375
-F 0 "J4" H 5075 4172 60  0000 C CNN
-F 1 "C64_User_Port" H 5075 4066 60  0000 C CNN
-F 2 "" H 4925 4075 60  0001 C CNN
-F 3 "~" H 4925 2175 60  0001 C CNN
-	1    5075 3375
+L c64_adapter_idc:C64_Modem_OUT J5
+U 1 1 62DCEDED
+P 5900 3900
+F 0 "J5" H 5912 4325 50  0000 C CNN
+F 1 "C64_Modem_IDC" H 5912 4234 50  0000 C CNN
+F 2 "BulkyModem:C64_Adapter_IDC" H 5925 3575 50  0001 C CNN
+F 3 "" H 5925 3575 50  0001 C CNN
+	1    5900 3900
 	1    0    0    -1
 $EndComp
-Text HLabel 6825 2525 2    50   Input ~ 0
-C64_TX
-Text HLabel 6825 3150 2    50   Input ~ 0
-C64_RTS
-Text HLabel 6825 3750 2    50   Output ~ 0
-C64_RX
-Text HLabel 6850 4375 2    50   Output ~ 0
-C64_CTS
-NoConn ~ 4425 2825
-NoConn ~ 4425 2925
-NoConn ~ 4425 3025
-NoConn ~ 4425 3125
-NoConn ~ 4425 3225
-NoConn ~ 4425 3325
-NoConn ~ 4425 3425
-NoConn ~ 4425 3525
-NoConn ~ 4425 3625
-NoConn ~ 4425 3725
-NoConn ~ 4425 3825
-NoConn ~ 4425 3925
-NoConn ~ 5725 2825
-NoConn ~ 5725 2925
-NoConn ~ 5725 3025
-NoConn ~ 5725 3125
-NoConn ~ 5725 3225
-NoConn ~ 5725 3325
-NoConn ~ 5725 3425
-NoConn ~ 5725 3525
-NoConn ~ 5725 3625
-NoConn ~ 5725 3725
-NoConn ~ 5725 3825
-NoConn ~ 5725 3925
+Wire Wire Line
+	6375 3700 6450 3700
+Wire Wire Line
+	6450 3700 6450 3800
+Wire Wire Line
+	6375 4100 6450 4100
+Connection ~ 6450 4100
+Wire Wire Line
+	6450 4100 6450 4175
+Wire Wire Line
+	6450 4000 6375 4000
+Connection ~ 6450 4000
+Wire Wire Line
+	6450 4000 6450 4100
+Wire Wire Line
+	6375 3900 6450 3900
+Connection ~ 6450 3900
+Wire Wire Line
+	6450 3900 6450 4000
+Wire Wire Line
+	6375 3800 6450 3800
+Connection ~ 6450 3800
+Wire Wire Line
+	6450 3800 6450 3900
+$Comp
+L power:GND #PWR0139
+U 1 1 62DD102B
+P 6450 4175
+F 0 "#PWR0139" H 6450 3925 50  0001 C CNN
+F 1 "GND" H 6455 4002 50  0000 C CNN
+F 2 "" H 6450 4175 50  0001 C CNN
+F 3 "" H 6450 4175 50  0001 C CNN
+	1    6450 4175
+	1    0    0    -1
+$EndComp
+Wire Wire Line
+	5450 3700 5375 3700
+Wire Wire Line
+	5375 3700 5375 3625
+$Comp
+L power:+5V #PWR?
+U 1 1 62DD613F
+P 5375 3625
+AR Path="/62DD613F" Ref="#PWR?"  Part="1"
+AR Path="/63AD1846/62DD613F" Ref="#PWR0140"  Part="1"
+F 0 "#PWR0140" H 5375 3475 50  0001 C CNN
+F 1 "+5V" H 5375 3800 50  0000 C CNN
+F 2 "" H 5375 3625 50  0001 C CNN
+F 3 "" H 5375 3625 50  0001 C CNN
+	1    5375 3625
+	1    0    0    -1
+$EndComp
+Wire Wire Line
+	5375 3800 5450 3800
+Wire Wire Line
+	5375 3900 5450 3900
+Wire Wire Line
+	5375 4000 5450 4000
+Wire Wire Line
+	5375 4100 5450 4100
 $EndSCHEMATC

Commit message: Add DCD
Connections:
- net GND: no longer J5.13 (GND)
- new net C64_DCD: J5.13 (GND)
Changed lines of the file:
@@
 	6450 3700 6450 3800
-Wire Wire Line
-	6375 4100 6450 4100
-Connection ~ 6450 4100
-Wire Wire Line
-	6450 4100 6450 4175
 Wire Wire Line
 	6450 4000 6375 4000
 Connection ~ 6450 4000
-Wire Wire Line
-	6450 4000 6450 4100
 Wire Wire Line
 	6375 3900 6450 3900
@@
 Wire Wire Line
 	5375 4100 5450 4100
+Text HLabel 6525 4100 2    50   Input ~ 0
+C64_DCD
+Wire Wire Line
+	6450 4000 6450 4175
+Wire Wire Line
+	6375 4100 6525 4100
 $EndSCHEMATC

Commit message: Initial layout
Parts:
- J5: footprint BulkyModem:C64_Adapter_IDC -> BulkyModem:UserPort_Adapter_IDC
Connections:
- net C64_DCD: now also J5.6 (DCD); no longer J5.13 (GND)
- net GND: now also J5.13 (GND), J5.14 (GND), J5.15 (GND)
- net C64_RI: now reaches J5.7 (RI)
Changed lines of the file:
@@
 F 0 "J5" H 5912 4325 50  0000 C CNN
 F 1 "C64_Modem_IDC" H 5912 4234 50  0000 C CNN
-F 2 "BulkyModem:C64_Adapter_IDC" H 5925 3575 50  0001 C CNN
+F 2 "BulkyModem:UserPort_Adapter_IDC" H 5925 3575 50  0001 C CNN
 F 3 "" H 5925 3575 50  0001 C CNN
 	1    5900 3900
@@
 	6450 3700 6450 3800
 Wire Wire Line
-	6450 4000 6375 4000
-Connection ~ 6450 4000
-Wire Wire Line
 	6375 3900 6450 3900
 Connection ~ 6450 3900
-Wire Wire Line
-	6450 3900 6450 4000
 Wire Wire Line
 	6375 3800 6450 3800
@@
 L power:GND #PWR0139
 U 1 1 62DD102B
-P 6450 4175
-F 0 "#PWR0139" H 6450 3925 50  0001 C CNN
-F 1 "GND" H 6455 4002 50  0000 C CNN
-F 2 "" H 6450 4175 50  0001 C CNN
-F 3 "" H 6450 4175 50  0001 C CNN
-	1    6450 4175
+P 6450 4450
+F 0 "#PWR0139" H 6450 4200 50  0001 C CNN
+F 1 "GND" H 6455 4277 50  0000 C CNN
+F 2 "" H 6450 4450 50  0001 C CNN
+F 3 "" H 6450 4450 50  0001 C CNN
+	1    6450 4450
 	1    0    0    -1
 $EndComp
@@
 Wire Wire Line
 	5375 4100 5450 4100
-Text HLabel 6525 4100 2    50   Input ~ 0
+Text HLabel 5375 4200 0    50   Input ~ 0
 C64_DCD
+Text HLabel 5375 4300 0    50   Input ~ 0
+C64_RI
 Wire Wire Line
-	6450 4000 6450 4175
+	5375 4200 5450 4200
 Wire Wire Line
-	6375 4100 6525 4100
+	5450 4300 5375 4300
+Wire Wire Line
+	6450 3900 6450 4000
+Wire Wire Line
+	6375 4000 6450 4000
+Connection ~ 6450 4000
+Wire Wire Line
+	6450 4000 6450 4100
+Wire Wire Line
+	6450 4100 6375 4100
+Connection ~ 6450 4100
+Wire Wire Line
+	6450 4100 6450 4200
+Wire Wire Line
+	6375 4200 6450 4200
+Connection ~ 6450 4200
+Wire Wire Line
+	6450 4200 6450 4300
+Wire Wire Line
+	6450 4300 6375 4300
+Connection ~ 6450 4300
+Wire Wire Line
+	6450 4300 6450 4450
 $EndSCHEMATC
