File: BulkyModem Module/audio_panel.kicad_sch (KiCad schematic)
At the start: 1 part

Commit message: Exported files
Changed lines of the file:
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@@
 	)
 	(global_label "AUDIO_RX"
-		(shape input)
+		(shape output)
 		(at 167.64 101.6 0)
 		(effects
@@
 	)
 	(global_label "AUDIO_TX"
-		(shape output)
+		(shape input)
 		(at 167.64 99.06 0)
 		(effects
