File: BulkyModem Module/c64_userport.kicad_sch (KiCad schematic)
At the start: 1 part, among them J5 C64_Modem_IDC

Commit message: Update project
Parts:
- J5: value C64_Modem_IDC -> C64_Modem_OUT
Changed lines of the file:
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@@
 			)
 		)
-		(property "Value" "C64_Modem_IDC"
+		(property "Value" "C64_Modem_OUT"
 			(at 150.1648 90.5764 0)
 			(effects
