File: BulkyModem UserPort Adapter/BulkyModem UserPort Adapter.sch (KiCad schematic (older format))
At the start: 7 parts, among them J1 C64_UserPort, J2 Temporary, J3 C64_Modem_IDC, M1 Mounting, M2 Mounting, M3 Mounting, M4 Mounting

Commit message: Add DCD
Connections:
- net GND: no longer J3.13 (GND)
- net at J2.12 (Pin_12): now also J3.13 (GND)
- no-connect marks 11 -> 10
Changed lines of the file:
@@
 $EndComp
 Wire Wire Line
-	8025 3575 8100 3575
+	8175 3575 8175 3675
+Connection ~ 8175 3875
+Connection ~ 8175 3775
 Wire Wire Line
-	8100 3575 8100 3675
+	8175 3775 8175 3875
+Connection ~ 8175 3675
 Wire Wire Line
-	8025 3975 8100 3975
-Connection ~ 8100 3975
-Wire Wire Line
-	8100 3975 8100 4050
-Wire Wire Line
-	8025 3875 8100 3875
-Connection ~ 8100 3875
-Wire Wire Line
-	8100 3875 8100 3975
-Wire Wire Line
-	8025 3775 8100 3775
-Connection ~ 8100 3775
-Wire Wire Line
-	8100 3775 8100 3875
-Wire Wire Line
-	8025 3675 8100 3675
-Connection ~ 8100 3675
-Wire Wire Line
-	8100 3675 8100 3775
+	8175 3675 8175 3775
 $Comp
 L power:GND #PWR0102
 U 1 1 62D9791D
-P 8100 4050
-F 0 "#PWR0102" H 8100 3800 50  0001 C CNN
-F 1 "GND" H 8105 3877 50  0000 C CNN
-F 2 "" H 8100 4050 50  0001 C CNN
-F 3 "" H 8100 4050 50  0001 C CNN
-	1    8100 4050
+P 8175 4125
+F 0 "#PWR0102" H 8175 3875 50  0001 C CNN
+F 1 "GND" H 8180 3952 50  0000 C CNN
+F 2 "" H 8175 4125 50  0001 C CNN
+F 3 "" H 8175 4125 50  0001 C CNN
+	1    8175 4125
 	1    0    0    -1
 $EndComp
@@
 NoConn ~ 5550 3575
 NoConn ~ 5550 3475
-$Comp
-L Connector_Generic:Conn_02x07_Odd_Even J2
-U 1 1 62DBC4D4
-P 6600 3875
-F 0 "J2" H 6650 4392 50  0000 C CNN
-F 1 "Temporary" H 6650 4301 50  0000 C CNN
-F 2 "Connector_PinHeader_2.54mm:PinHeader_2x07_P2.54mm_Vertical" H 6600 3875 50  0001 C CNN
-F 3 "~" H 6600 3875 50  0001 C CNN
-	1    6600 3875
-	1    0    0    -1
-$EndComp
 Wire Wire Line
 	6900 3575 6975 3575
@@
 Text GLabel 6325 4075 0    50   Output ~ 0
 DCD
-NoConn ~ 6900 4075
 Wire Wire Line
 	6325 4075 6400 4075
@@
 	6225 3500 6325 3500
 Connection ~ 6325 3500
+$Comp
+L Connector_Generic:Conn_02x07_Odd_Even J2
+U 1 1 62DBC4D4
+P 6600 3875
+F 0 "J2" H 6650 4392 50  0000 C CNN
+F 1 "Temporary" H 6650 4301 50  0000 C CNN
+F 2 "Connector_PinHeader_2.54mm:PinHeader_2x07_P2.54mm_Vertical" H 6600 3875 50  0001 C CNN
+F 3 "~" H 6600 3875 50  0001 C CNN
+	1    6600 3875
+	1    0    0    -1
+$EndComp
+Wire Wire Line
+	6900 4075 8100 4075
+Wire Wire Line
+	8100 4075 8100 3975
+Wire Wire Line
+	8100 3975 8025 3975
+Wire Wire Line
+	8025 3875 8175 3875
+Wire Wire Line
+	8025 3775 8175 3775
+Wire Wire Line
+	8025 3575 8175 3575
+Wire Wire Line
+	8025 3675 8175 3675
+Wire Wire Line
+	8175 3875 8175 4125
 $EndSCHEMATC

Commit message: Changed IDC pin count
Parts:
- J2: footprint Connector_PinHeader_2.54mm:PinHeader_2x07_P2.54mm_Vertical -> Connector_PinHeader_2.54mm:PinHeader_2x08_P2.54mm_Vertical; symbol Connector_Generic:Conn_02x07_Odd_Even -> Connector_Generic:Conn_02x08_Odd_Even
- J3: footprint BulkyModem:C64_Adapter_IDC -> BulkyModem:UserPort_Adapter_IDC
Connections:
- net GND: now also J2.15 (Pin_15), J2.16 (Pin_16), J3.13 (GND), J3.14 (GND), J3.15 (GND); no longer J2.13 (Pin_13), J2.14 (Pin_14)
- net RI: now reaches J1.F (PB3)
- net RI: now also J2.13 (Pin_13)
- net at J2.12 (Pin_12): now also J3.6 (DCD); no longer J3.13 (GND)
- net at J3.7 (RI): now also J2.14 (Pin_14)
- no-connect marks 10 -> 9
Changed lines of the file:
@@
 F 0 "J3" H 7562 4200 50  0000 C CNN
 F 1 "C64_Modem_IDC" H 7562 4109 50  0000 C CNN
-F 2 "BulkyModem:C64_Adapter_IDC" H 7575 3450 50  0001 C CNN
+F 2 "BulkyModem:UserPort_Adapter_IDC" H 7575 3450 50  0001 C CNN
 F 3 "" H 7575 3450 50  0001 C CNN
 	1    7550 3775
@@
 L power:GND #PWR0102
 U 1 1 62D9791D
-P 8175 4125
-F 0 "#PWR0102" H 8175 3875 50  0001 C CNN
-F 1 "GND" H 8180 3952 50  0000 C CNN
-F 2 "" H 8175 4125 50  0001 C CNN
-F 3 "" H 8175 4125 50  0001 C CNN
-	1    8175 4125
+P 8175 4325
+F 0 "#PWR0102" H 8175 4075 50  0001 C CNN
+F 1 "GND" H 8180 4152 50  0000 C CNN
+F 2 "" H 8175 4325 50  0001 C CNN
+F 3 "" H 8175 4325 50  0001 C CNN
+	1    8175 4325
 	1    0    0    -1
 $EndComp
@@
 	4025 4075 4250 4075
 NoConn ~ 4250 3675
-NoConn ~ 4250 3775
 NoConn ~ 4250 3975
 NoConn ~ 5550 4075
@@
 	6900 3975 7100 3975
 Wire Wire Line
-	6900 4175 6975 4175
-Wire Wire Line
-	6975 4175 6975 4250
+	6900 4275 6975 4275
 $Comp
 L power:GND #PWR0103
 U 1 1 62DCE03D
-P 6975 4325
-F 0 "#PWR0103" H 6975 4075 50  0001 C CNN
-F 1 "GND" H 6980 4152 50  0000 C CNN
-F 2 "" H 6975 4325 50  0001 C CNN
-F 3 "" H 6975 4325 50  0001 C CNN
-	1    6975 4325
+P 6975 4425
+F 0 "#PWR0103" H 6975 4175 50  0001 C CNN
+F 1 "GND" H 6980 4252 50  0000 C CNN
+F 2 "" H 6975 4425 50  0001 C CNN
+F 3 "" H 6975 4425 50  0001 C CNN
+	1    6975 4425
 	1    0    0    -1
 $EndComp
@@
 	6325 4075 6400 4075
 Wire Wire Line
-	6400 4175 6325 4175
-Wire Wire Line
-	6325 4175 6325 4250
-Wire Wire Line
-	6325 4250 6975 4250
-Connection ~ 6975 4250
-Wire Wire Line
-	6975 4325 6975 4250
+	6400 4275 6325 4275
+Wire Wire Line
+	6325 4275 6325 4350
+Wire Wire Line
+	6325 4350 6975 4350
 Wire Wire Line
 	6400 3575 6325 3575
@@
 Wire Wire Line
 	6975 3500 6975 3575
-Text Notes 6275 4675 0    50   ~ 0
+Text Notes 6075 4475 0    50   ~ 0
 Connect DCD to RTS?
 Text GLabel 5800 3675 2    50   Input ~ 0
@@
 Connection ~ 6325 3500
 $Comp
-L Connector_Generic:Conn_02x07_Odd_Even J2
+L Connector_Generic:Conn_02x08_Odd_Even J2
 U 1 1 62DBC4D4
 P 6600 3875
 F 0 "J2" H 6650 4392 50  0000 C CNN
 F 1 "Temporary" H 6650 4301 50  0000 C CNN
-F 2 "Connector_PinHeader_2.54mm:PinHeader_2x07_P2.54mm_Vertical" H 6600 3875 50  0001 C CNN
+F 2 "Connector_PinHeader_2.54mm:PinHeader_2x08_P2.54mm_Vertical" H 6600 3875 50  0001 C CNN
 F 3 "~" H 6600 3875 50  0001 C CNN
 	1    6600 3875
@@
 $EndComp
 Wire Wire Line
-	6900 4075 8100 4075
-Wire Wire Line
-	8100 4075 8100 3975
-Wire Wire Line
-	8100 3975 8025 3975
-Wire Wire Line
 	8025 3875 8175 3875
 Wire Wire Line
@@
 	8025 3675 8175 3675
 Wire Wire Line
-	8175 3875 8175 4125
+	6900 4075 7100 4075
+Wire Wire Line
+	6975 4350 6975 4425
+Wire Wire Line
+	6975 4275 6975 4350
+Connection ~ 6975 4350
+Wire Wire Line
+	7100 4175 6900 4175
+Text GLabel 6325 4175 0    50   Output ~ 0
+RI
+Wire Wire Line
+	6325 4175 6400 4175
+Text GLabel 4025 3775 0    50   Input ~ 0
+RI
+Wire Wire Line
+	4250 3775 4025 3775
+Wire Wire Line
+	8175 3875 8175 3975
+Wire Wire Line
+	8025 4175 8175 4175
+Connection ~ 8175 4175
+Wire Wire Line
+	8175 4175 8175 4325
+Wire Wire Line
+	8025 4075 8175 4075
+Connection ~ 8175 4075
+Wire Wire Line
+	8175 4075 8175 4175
+Wire Wire Line
+	8025 3975 8175 3975
+Connection ~ 8175 3975
+Wire Wire Line
+	8175 3975 8175 4075
 $EndSCHEMATC

Commit message: Changed C64 UserPort adapter schematic
Parts:
- removed J2: Temporary, Connector_PinHeader_2.54mm:PinHeader_2x08_P2.54mm_Vertical, symbol Connector_Generic:Conn_02x08_Odd_Even
- added JP1, JP2: UP9600, symbol Jumper:SolderJumper_2_Bridged
- J1: symbol c64_user_port:C64_User_Port -> c64_user_port:C64_User_Port_Serial
Connections:
- net CTS: now also J3.5 (CTS)
- net DCD: now also J3.6 (DCD)
- net RI: now also J3.7 (RI)
- net RTS: now also J3.4 (RTS)
- net TXD: now reaches J3.2 (TX)
- net TXD: now also J1.B (~FLAG2), J1.C (PB0(RXD)), JP2.2 (B)
- net RXD: now reaches J3.3 (RX)
- net RXD: now also J1.M (PA2(TXD)), JP1.2 (B)
- net RX: no longer names the net of J1.5 (SP1)
- net RX: now also JP1.1 (A); no longer J1.M (PA2)
- removed net TX: J1.7 (SP2), J1.B (~FLAG2), J1.C (PB0)
- new net: J1.7 (SP2), JP2.1 (A)
- no-connect marks 9 -> 10
Other:
- note added: "UP9600 is not compatible with burst mode disk drives\nconnected to Commodore 128, as UP9600 uses the HW\ntimers for serial."
- note removed: "Connect DCD to RTS?"
- moved on the sheet: J1, J3

Commit message: Alternate panel designs
Parts:
- JP1, JP2: footprint (none) -> solder_bridge:bridge
Changed lines of the file:
@@
 F 0 "JP1" H 5425 3855 50  0000 C CNN
 F 1 "UP9600" H 5425 3764 50  0000 C CNN
-F 2 "" H 5425 3650 50  0001 C CNN
+F 2 "solder_bridge:bridge" H 5425 3650 50  0001 C CNN
 F 3 "~" H 5425 3650 50  0001 C CNN
 	1    5425 3650
@@
 F 0 "JP2" H 5425 3725 50  0000 C CNN
 F 1 "UP9600" H 5425 3650 50  0000 C CNN
-F 2 "" H 5425 3850 50  0001 C CNN
+F 2 "solder_bridge:bridge" H 5425 3850 50  0001 C CNN
 F 3 "~" H 5425 3850 50  0001 C CNN
 	1    5425 3850

Commit message: Updated UserPort layout
Parts:
- JP1, JP2: footprint solder_bridge:bridge -> Connector_PinHeader_2.54mm:PinHeader_1x02_P2.54mm_Vertical
Changed lines of the file:
@@
 F 0 "JP1" H 5425 3855 50  0000 C CNN
 F 1 "UP9600" H 5425 3764 50  0000 C CNN
-F 2 "solder_bridge:bridge" H 5425 3650 50  0001 C CNN
+F 2 "Connector_PinHeader_2.54mm:PinHeader_1x02_P2.54mm_Vertical" H 5425 3650 50  0001 C CNN
 F 3 "~" H 5425 3650 50  0001 C CNN
 	1    5425 3650
@@
 F 0 "JP2" H 5425 3725 50  0000 C CNN
 F 1 "UP9600" H 5425 3650 50  0000 C CNN
-F 2 "solder_bridge:bridge" H 5425 3850 50  0001 C CNN
+F 2 "Connector_PinHeader_2.54mm:PinHeader_1x02_P2.54mm_Vertical" H 5425 3850 50  0001 C CNN
 F 3 "~" H 5425 3850 50  0001 C CNN
 	1    5425 3850

Commit message: Export files
Other:
- note added: "UP9600 is not compatible with burst mode disk drives\nconnected to Commodore 128. This is due to UP9600\nusing HW-timers that are needed for other things on\nthe 128."
- note removed: "UP9600 is not compatible with burst mode disk drives\nconnected to Commodore 128, as UP9600 uses the HW\ntimers for serial."
Changed lines of the file:
@@
 Comment2 ""
 Comment3 ""
-Comment4 "UserPort adapter for connecting to the BulkyModem via a 2x5 pin IDC cable."
+Comment4 "UserPort adapter for connecting to the BulkyModem via a 2x8-pin IDC cable."
 $EndDescr
 $Comp
@@
 Wire Wire Line
 	5575 3850 5650 3850
-Text Notes 5275 4425 0    50   ~ 0
-UP9600 is not compatible with burst mode disk drives\nconnected to Commodore 128, as UP9600 uses the HW\ntimers for serial.
+Text Notes 5275 4500 0    50   ~ 0
+UP9600 is not compatible with burst mode disk drives\nconnected to Commodore 128. This is due to UP9600\nusing HW-timers that are needed for other things on\nthe 128.
 $EndSCHEMATC
