File: BulkyModem Module Panel B/BulkyModem Module Panel B.sch (KiCad schematic (older format))
At the start: 20 parts, among them J1 Front Panel, M1 Mounting_Pin, M2 Mounting_Pin, M3 Mounting_Pin, M4 Mounting_Pin, SW1 MODE, SW2 POW

Commit message: Tweaks needed to make revision C actually work.
Parts:
- D17: symbol Device:LED_RGBC -> led_rgbc:LED_RGBC
Connections:
- net GND: now also D17.2 (K); no longer D17.4 (K)
- net at R2.2: now also D17.3 (GA); no longer D17.2 (GA)
Changed lines of the file:
@@
 NoConn ~ 9025 2725
-$Comp
-L Device:LED_RGBC D17
-U 1 1 6434C68B
-P 2800 3325
-F 0 "D17" V 2846 2995 50  0000 R CNN
-F 1 "LED_RGBC" V 2755 2995 50  0000 R CNN
-F 2 "LED_THT:LED_D5.0mm-4_RGB_Wide_Pins" H 2800 3275 50  0001 C CNN
-F 3 "~" H 2800 3275 50  0001 C CNN
-	1    2800 3325
-	0    -1   -1   0
-$EndComp
 $Comp
 L power:GND #PWR0109
@@
 Wire Bus Line
 	8275 2725 8275 3625
+$Comp
+L led_rgbc:LED_RGBC D17
+U 1 1 6434C68B
+P 2800 3325
+F 0 "D17" V 2846 2995 50  0000 R CNN
+F 1 "LED_RGBC" V 2755 2995 50  0000 R CNN
+F 2 "LED_THT:LED_D5.0mm-4_RGB_Wide_Pins" H 2800 3275 50  0001 C CNN
+F 3 "~" H 2800 3275 50  0001 C CNN
+	1    2800 3325
+	0    -1   -1   0
+$EndComp
 $EndSCHEMATC
