File: faceplates/BulkyModem FP3/BulkyModem FP3.kicad_pcb (KiCad board)
At the start: 2 copper layers, 100 x 35 mm, 5 parts, among them M1 Mounting_Pin, M2 Mounting_Pin, M3 Mounting_Pin, M4 Mounting_Pin

Commit message: Exported files
Other:
- outline, holes or cut-outs redrawn
- board text added: "BulkyModem Front Panel FP3 (rev. B) github.com/tebl"
- board text removed: "BulkyModem Front Panel FP3 (rev. A) github.com/tebl"
