File: faceplates/BulkyModem Terminal FP3/BulkyModem Terminal FP3.kicad_pcb (KiCad board)
At the start: 2 copper layers, 100 x 35 mm, 5 parts, among them M1 Mounting_Pin, M2 Mounting_Pin, M3 Mounting_Pin, M4 Mounting_Pin

Commit message: TTL legend
Other:
- outline, holes or cut-outs redrawn
- board text added: "+ VCC"
- board text added: "- GND"
- board text added: "< RTS"
- board text added: "< TxD"
- board text added: "> CTS"
- board text added: "> RxD"

Commit message: Exported files
Changed lines of the file:
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@@
 			)
 		)
-		(attr through_hole)
+		(attr through_hole board_only exclude_from_pos_files exclude_from_bom allow_missing_courtyard)
 		(fp_poly
 			(pts
@@
 		)
 	)
-	(gr_text "TX"
+	(gr_text "RX"
 		(at 115.055 119.928 0)
 		(layer "F.SilkS")
@@
 			)
 		)
-		(render_cache "TX" 0
-			(polygon
-				(pts
-					(xy 114.183297 120.343) (xy 114.183297 119.298861) (xy 113.829878 119.298861) (xy 113.829878 119.123739)
-					(xy 114.877191 119.123739) (xy 114.877191 119.298861) (xy 114.533297 119.298861) (xy 114.533297 120.343)
+		(render_cache "RX" 0
+			(polygon
+				(pts
+					(xy 114.705244 119.295686) (xy 114.877191 119.295686) (xy 114.877191 119.63958) (xy 114.705244 119.63958)
+					(xy 114.705244 119.811527) (xy 114.529878 119.811527) (xy 114.529878 119.983474) (xy 114.705244 119.983474)
+					(xy 114.705244 120.167877) (xy 114.877191 120.167877) (xy 114.877191 120.343) (xy 114.529878 120.343)
+					(xy 114.529878 120.167877) (xy 114.355244 120.167877) (xy 114.355244 119.983474) (xy 114.179878 119.983474)
+					(xy 114.179878 120.343) (xy 113.829878 120.343) (xy 113.829878 119.63958) (xy 114.179878 119.63958)
+					(xy 114.529878 119.63958) (xy 114.529878 119.298861) (xy 114.179878 119.298861) (xy 114.179878 119.63958)
+					(xy 113.829878 119.63958) (xy 113.829878 119.123739) (xy 114.705244 119.123739)
 				)
 			)
@@
 		)
 	)
-	(gr_text "CTS"
+	(gr_text "RTS"
 		(at 122.04 119.928 0)
 		(layer "F.SilkS")
@@
 			)
 		)
-		(render_cache "CTS" 0
-			(polygon
-				(pts
-					(xy 120.374263 120.343) (xy 120.374263 120.167877) (xy 120.202317 120.167877) (xy 120.202317 119.295686)
-					(xy 120.374263 119.295686) (xy 120.374263 119.123739) (xy 121.077683 119.123739) (xy 121.077683 119.295686)
-					(xy 121.24963 119.295686) (xy 121.24963 119.470808) (xy 120.89963 119.470808) (xy 120.89963 119.298861)
-					(xy 120.552317 119.298861) (xy 120.552317 120.167877) (xy 120.89963 120.167877) (xy 120.89963 119.99593)
-					(xy 121.24963 119.99593) (xy 121.24963 120.167877) (xy 121.077683 120.167877) (xy 121.077683 120.343)
+		(render_cache "RTS" 0
+			(polygon
+				(pts
+					(xy 121.077683 119.295686) (xy 121.24963 119.295686) (xy 121.24963 119.63958) (xy 121.077683 119.63958)
+					(xy 121.077683 119.811527) (xy 120.902317 119.811527) (xy 120.902317 119.983474) (xy 121.077683 119.983474)
+					(xy 121.077683 120.167877) (xy 121.24963 120.167877) (xy 121.24963 120.343) (xy 120.902317 120.343)
+					(xy 120.902317 120.167877) (xy 120.727683 120.167877) (xy 120.727683 119.983474) (xy 120.552317 119.983474)
+					(xy 120.552317 120.343) (xy 120.202317 120.343) (xy 120.202317 119.63958) (xy 120.552317 119.63958)
+					(xy 120.902317 119.63958) (xy 120.902317 119.298861) (xy 120.552317 119.298861) (xy 120.552317 119.63958)
+					(xy 120.202317 119.63958) (xy 120.202317 119.123739) (xy 121.077683 119.123739)
 				)
 			)
@@
 		)
 	)
-	(gr_text "RX"
+	(gr_text "TX"
 		(at 108.07 119.928 0)
 		(layer "F.SilkS")
@@
 			)
 		)
-		(render_cache "RX" 0
-			(polygon
-				(pts
-					(xy 107.720244 119.295686) (xy 107.892191 119.295686) (xy 107.892191 119.63958) (xy 107.720244 119.63958)
-					(xy 107.720244 119.811527) (xy 107.544878 119.811527) (xy 107.544878 119.983474) (xy 107.720244 119.983474)
-					(xy 107.720244 120.167877) (xy 107.892191 120.167877) (xy 107.892191 120.343) (xy 107.544878 120.343)
-					(xy 107.544878 120.167877) (xy 107.370244 120.167877) (xy 107.370244 119.983474) (xy 107.194878 119.983474)
-					(xy 107.194878 120.343) (xy 106.844878 120.343) (xy 106.844878 119.63958) (xy 107.194878 119.63958)
-					(xy 107.544878 119.63958) (xy 107.544878 119.298861) (xy 107.194878 119.298861) (xy 107.194878 119.63958)
-					(xy 106.844878 119.63958) (xy 106.844878 119.123739) (xy 107.720244 119.123739)
+		(render_cache "TX" 0
+			(polygon
+				(pts
+					(xy 107.198297 120.343) (xy 107.198297 119.298861) (xy 106.844878 119.298861) (xy 106.844878 119.123739)
+					(xy 107.892191 119.123739) (xy 107.892191 119.298861) (xy 107.548297 119.298861) (xy 107.548297 120.343)
 				)
 			)
@@
 		)
 	)
-	(gr_text "RTS"
+	(gr_text "CTS"
 		(at 129.025 119.928 0)
 		(layer "F.SilkS")
@@
 			)
 		)
-		(render_cache "RTS" 0
-			(polygon
-				(pts
-					(xy 128.062683 119.295686) (xy 128.23463 119.295686) (xy 128.23463 119.63958) (xy 128.062683 119.63958)
-					(xy 128.062683 119.811527) (xy 127.887317 119.811527) (xy 127.887317 119.983474) (xy 128.062683 119.983474)
-					(xy 128.062683 120.167877) (xy 128.23463 120.167877) (xy 128.23463 120.343) (xy 127.887317 120.343)
-					(xy 127.887317 120.167877) (xy 127.712683 120.167877) (xy 127.712683 119.983474) (xy 127.537317 119.983474)
-					(xy 127.537317 120.343) (xy 127.187317 120.343) (xy 127.187317 119.63958) (xy 127.537317 119.63958)
-					(xy 127.887317 119.63958) (xy 127.887317 119.298861) (xy 127.537317 119.298861) (xy 127.537317 119.63958)
-					(xy 127.187317 119.63958) (xy 127.187317 119.123739) (xy 128.062683 119.123739)
-				)
-			)
+		(render_cache "CTS" 0
+			(polygon
+				(pts
+					(xy 127.359263 120.343) (xy 127.359263 120.167877) (xy 127.187317 120.167877) (xy 127.187317 119.295686)
+					(xy 127.359263 119.295686) (xy 127.359263 119.123739) (xy 128.062683 119.123739) (xy 128.062683 119.295686)
+					(xy 128.23463 119.295686) (xy 128.23463 119.470808) (xy 127.88463 119.470808) (xy 127.88463 119.298861)
+					(xy 127.537317 119.298861) (xy 127.537317 120.167877) (xy 127.88463 120.167877) (xy 127.88463 119.99593)
+					(xy 128.23463 119.99593) (xy 128.23463 120.167877) (xy 128.062683 120.167877) (xy 128.062683 120.343)
+				)
+			)
