File: faceplates/BulkyModem Terminal FP3/BulkyModem Terminal FP3.kicad_sch (KiCad schematic)
At the start: 4 parts, among them M1 Mounting_Pin, M2 Mounting_Pin, M3 Mounting_Pin, M4 Mounting_Pin

Commit message: Move PS/2 port to the back with some caveats, basically needs a custom top panel
Other:
- title: BulkyModem Front Plate (FP3) -> BulkyModem Terminal (FP3)
Changed lines of the file:
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@@
 	(paper "A4")
 	(title_block
-		(title "BulkyModem Front Plate (FP3)")
+		(title "BulkyModem Terminal (FP3)")
 		(rev "A")
-		(comment 2 "Faceplate that extends down past the main board.")
+		(comment 2 "Faceplate that extends down past the main board, specific for the terminal.")
 		(comment 4 "A cosmetic plate to go on the front of the device.")
 	)
@@
 		)
 		(instances
-			(project "BulkyModem FP3"
+			(project "BulkyModem Terminal FP3"
 				(path "/7d1c5d90-76e9-4eed-88d7-b688de928396"
 					(reference "M1")
@@
 		)
 		(instances
-			(project "BulkyModem FP3"
+			(project "BulkyModem Terminal FP3"
 				(path "/7d1c5d90-76e9-4eed-88d7-b688de928396"
 					(reference "M2")
@@
 		)
 		(instances
-			(project "BulkyModem FP3"
+			(project "BulkyModem Terminal FP3"
 				(path "/7d1c5d90-76e9-4eed-88d7-b688de928396"
 					(reference "M3")
@@
 		)
 		(instances
-			(project "BulkyModem FP3"
+			(project "BulkyModem Terminal FP3"
 				(path "/7d1c5d90-76e9-4eed-88d7-b688de928396"
 					(reference "M4")
@@
 		)
 		(instances
-			(project "BulkyModem FP3"
+			(project "BulkyModem Terminal FP3"
 				(path "/7d1c5d90-76e9-4eed-88d7-b688de928396"
 					(reference "#PWR0111")
@@
 		)
 		(instances
-			(project "BulkyModem FP3"
+			(project "BulkyModem Terminal FP3"
 				(path "/7d1c5d90-76e9-4eed-88d7-b688de928396"
 					(reference "#FLG?")
