File: BulkyModem-32 Mini/front_panel.kicad_sch (KiCad schematic)
At the start: 10 parts

Commit message: ESP32 Mini cleanup
Other:
- note added: "Resistor values have been picked from a hat. If it already has a colour without applying power, then you should pick something lower. Generally, you should consider datasheets when selecting and then calculating an appropriate value. Or just go with the one suggested and change them out later."
- title: BulkyModem Module (Front Panel) -> BulkyModem-32 Mini (Front Panel)
- moved on the sheet: D1, D2, D3, D4, D5, R1, R2, R3, R4, R6
