File: BulkyModem-32 Mini/power.kicad_sch (KiCad schematic)
At the start: 3 parts, among them U6 74HCT32

Commit message: ESP32 Mini cleanup
Other:
- note added: "The Mini boards are powered from USB, so there's not much interesting to actually see here."
- title: BulkyModem Module (Power) -> BulkyModem-32 Mini (Power)
- moved on the sheet: C1, C8, U6E
Changed lines of the file:
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@@
 	(paper "A4")
 	(title_block
-		(title "BulkyModem Module (Power)")
+		(title "BulkyModem-32 Mini (Power)")
 	)
 	(junction
-		(at 189.23 106.68)
+		(at 157.48 110.49)
 		(diameter 0)
 		(color 0 0 0 0)
@@
 	)
 	(junction
-		(at 109.22 106.68)
+		(at 142.24 110.49)
 		(diameter 0)
 		(color 0 0 0 0)
 	)
 	(junction
-		(at 109.22 77.47)
+		(at 142.24 81.28)
 		(diameter 0)
 		(color 0 0 0 0)
 	)
 	(junction
-		(at 97.79 77.47)
+		(at 130.81 81.28)
 		(diameter 0)
 		(color 0 0 0 0)
@@
 	(wire
 		(pts
-			(xy 109.22 77.47) (xy 109.22 88.9)
-		)
-		(stroke
-			(width 0)
-			(type default)
-		)
-	)
-	(wire
-		(pts
-			(xy 97.79 77.47) (xy 97.79 88.9)
-		)
-		(stroke
-			(width 0)
-			(type default)
-		)
-	)
-	(wire
-		(pts
-			(xy 97.79 93.98) (xy 97.79 106.68)
-		)
-		(stroke
-			(width 0)
-			(type default)
-		)
-	)
-	(wire
-		(pts
-			(xy 97.79 74.93) (xy 97.79 77.47)
+			(xy 142.24 81.28) (xy 142.24 92.71)
+		)
+		(stroke
+			(width 0)
+			(type default)
+		)
+	)
+	(wire
+		(pts
+			(xy 130.81 81.28) (xy 130.81 92.71)
+		)
+		(stroke
+			(width 0)
+			(type default)
+		)
+	)
+	(wire
+		(pts
+			(xy 130.81 97.79) (xy 130.81 110.49)
+		)
+		(stroke
+			(width 0)
+			(type default)
+		)
+	)
+	(wire
+		(pts
+			(xy 130.81 81.28) (xy 142.24 81.28)
+		)
+		(stroke
+			(width 0)
+			(type default)
+		)
+	)
+	(wire
+		(pts
+			(xy 142.24 110.49) (xy 157.48 110.49)
+		)
+		(stroke
+			(width 0)
+			(type default)
+		)
+	)
+	(wire
+		(pts
+			(xy 130.81 78.74) (xy 130.81 81.28)
 		)
 		(stroke
@@
 	(wire
 		(pts
-			(xy 189.23 107.95) (xy 189.23 106.68)
+			(xy 157.48 111.76) (xy 157.48 110.49)
 		)
 		(stroke
@@
 	(wire
 		(pts
-			(xy 97.79 106.68) (xy 109.22 106.68)
-		)
-		(stroke
-			(width 0)
-			(type default)
-		)
-	)
-	(wire
-		(pts
-			(xy 109.22 77.47) (xy 189.23 77.47)
-		)
-		(stroke
-			(width 0)
-			(type default)
-		)
-	)
-	(wire
-		(pts
-			(xy 189.23 77.47) (xy 189.23 78.74)
-		)
-		(stroke
-			(width 0)
-			(type default)
-		)
-	)
-	(wire
-		(pts
-			(xy 189.23 104.14) (xy 189.23 106.68)
-		)
-		(stroke
-			(width 0)
-			(type default)
-		)
-	)
-	(wire
-		(pts
-			(xy 97.79 77.47) (xy 109.22 77.47)
+			(xy 130.81 110.49) (xy 142.24 110.49)
+		)
+		(stroke
+			(width 0)
+			(type default)
+		)
+	)
+	(wire
+		(pts
+			(xy 157.48 81.28) (xy 157.48 82.55)
+		)
+		(stroke
+			(width 0)
+			(type default)
+		)
+	)
+	(wire
+		(pts
+			(xy 157.48 107.95) (xy 157.48 110.49)
 		)
 		(stroke
@@
 	(wire
 		(pts
-			(xy 109.22 93.98) (xy 109.22 106.68)
-		)
-		(stroke
-			(width 0)
-			(type default)
-		)
-	)
-	(wire
-		(pts
-			(xy 109.22 106.68) (xy 189.23 106.68)
+			(xy 142.24 97.79) (xy 142.24 110.49)
 		)
 		(stroke
@@
 			(width 0)
 			(type default)
+		)
+	)
+	(wire
+		(pts
+			(xy 142.24 81.28) (xy 157.48 81.28)
+		)
+		(stroke
+			(width 0)
+			(type default)
+		)
+	)
+	(text "The Mini boards are powered from USB,\nso there's not much interesting to\nactually see here."
+		(exclude_from_sim no)
+		(at 190.5 95.25 0)
+		(effects
+			(font
+				(size 1.27 1.27)
+			)
 		)
 	)
@@
 	(symbol
 		(lib_id "power:+5V")
-		(at 97.79 74.93 0)
+		(at 130.81 78.74 0)
 		(unit 1)
 		(exclude_from_sim no)
@@
 		(dnp no)
 		(property "Reference" "#PWR0110"
-			(at 97.79 78.74 0)
+			(at 130.81 82.55 0)
 			(effects
 				(font
@@
 		)
 		(property "Value" "+5V"
-			(at 97.79 71.374 0)
+			(at 130.81 75.184 0)
 			(effects
 				(font
@@
 		)
 		(property "Footprint" ""
-			(at 97.79 74.93 0)
+			(at 130.81 78.74 0)
 			(effects
 				(font
@@
 		)
 		(property "Datasheet" ""
-			(at 97.79 74.93 0)
+			(at 130.81 78.74 0)
 			(effects
 				(font
@@
 		)
 		(property "Description" "Power symbol creates a global label with name \"+5V\""
-			(at 97.79 74.93 0)
+			(at 130.81 78.74 0)
 			(effects
 				(font
@@
 	(symbol
 		(lib_id "power:GND")
-		(at 189.23 107.95 0)
+		(at 157.48 111.76 0)
 		(unit 1)
 		(exclude_from_sim no)
@@
 		(dnp no)
 		(property "Reference" "#PWR0133"
-			(at 189.23 114.3 0)
+			(at 157.48 118.11 0)
 			(effects
 				(font
@@
 		)
 		(property "Value" "GND"
-			(at 189.357 112.3442 0)
+			(at 157.607 116.1542 0)
 			(effects
 				(font
@@
 		)
 		(property "Footprint" ""
-			(at 189.23 107.95 0)
+			(at 157.48 111.76 0)
 			(effects
 				(font
@@
 		)
 		(property "Datasheet" ""
-			(at 189.23 107.95 0)
+			(at 157.48 111.76 0)
 			(effects
 				(font
@@
 		)
 		(property "Description" "Power symbol creates a global label with name \"GND\" , ground"
-			(at 189.23 107.95 0)
+			(at 157.48 111.76 0)
 			(effects
 				(font
@@
 	(symbol
 		(lib_id "74xx:74LS32")
-		(at 189.23 91.44 0)
+		(at 157.48 95.25 0)
 		(unit 5)
 		(exclude_from_sim no)
@@
 		(dnp no)
 		(property "Reference" "U6"
-			(at 189.23 90.17 0)
+			(at 157.48 93.98 0)
 			(effects
 				(font
@@
 		)
 		(property "Value" "74HCT32"
-			(at 189.23 92.71 0)
+			(at 157.48 96.52 0)
 			(effects
 				(font
@@
 		)
 		(property "Footprint" "Package_DIP:DIP-14_W7.62mm_Socket_LongPads"
-			(at 189.23 91.44 0)
+			(at 157.48 95.25 0)
 			(effects
 				(font
@@
 		)
 		(property "Datasheet" "http://www.ti.com/lit/gpn/sn74LS32"
-			(at 189.23 91.44 0)
+			(at 157.48 95.25 0)
 			(effects
 				(font
@@
 		)
 		(property "Description" "Quad 2-input OR"
-			(at 189.23 91.44 0)
+			(at 157.48 95.25 0)
 			(effects
 				(font
@@
 	(symbol
 		(lib_id "Device:C_Small")
-		(at 97.79 91.44 0)
+		(at 130.81 95.25 0)
 		(unit 1)
 		(exclude_from_sim no)
@@
 		(dnp no)
 		(property "Reference" "C8"
-			(at 100.1268 90.2716 0)
+			(at 133.1468 94.0816 0)
 			(effects
 				(font
@@
 		)
 		(property "Value" "100nF"
-			(at 100.1268 92.583 0)
+			(at 133.1468 96.393 0)
 			(effects
 				(font
@@
 		)
 		(property "Footprint" "Capacitor_THT:C_Disc_D4.7mm_W2.5mm_P5.00mm"
-			(at 97.79 91.44 0)
+			(at 130.81 95.25 0)
 			(effects
 				(font
@@
 		)
 		(property "Datasheet" "~"
-			(at 97.79 91.44 0)
+			(at 130.81 95.25 0)
 			(effects
 				(font
@@
 		)
 		(property "Description" "Unpolarized capacitor, small symbol"
-			(at 97.79 91.44 0)
+			(at 130.81 95.25 0)
 			(effects
 				(font
@@
 	(symbol
 		(lib_id "Device:C_Small")
-		(at 109.22 91.44 0)
+		(at 142.24 95.25 0)
 		(unit 1)
 		(exclude_from_sim no)
@@
 		(dnp no)
 		(property "Reference" "C1"
-			(at 111.5568 90.2716 0)
+			(at 144.5768 94.0816 0)
 			(effects
 				(font
@@
 		)
 		(property "Value" "100nF"
-			(at 111.5568 92.583 0)
+			(at 144.5768 96.393 0)
 			(effects
 				(font
@@
 		)
 		(property "Footprint" "Capacitor_THT:C_Disc_D4.7mm_W2.5mm_P5.00mm"
-			(at 109.22 91.44 0)
+			(at 142.24 95.25 0)
 			(effects
 				(font
@@
 		)
 		(property "Datasheet" "~"
-			(at 109.22 91.44 0)
+			(at 142.24 95.25 0)
 			(effects
 				(font
@@
 		)
 		(property "Description" "Unpolarized capacitor, small symbol"
-			(at 109.22 91.44 0)
-			(effects
-				(font
+			(at 142.24 95.25 0)
+			(effects
+				(font
