File: BulkyModem-32 Mini/rs232.kicad_sch (KiCad schematic)
At the start: 6 parts, among them J2 DCE, U3 MAX232

Commit message: ESP32 Mini cleanup
Other:
- note added: "C2-C5 must be electrolytic 1uF when using older or cheaper MAX232 variants, these can be replaced with standard 100nF when used with the MAX232A."
- note added: "I know that there are 3.3v versions of these chips available, but as I regularly work with 5v - those are the chips that I have available. Besides, there are lots of bad cloned chips and I accidentally lost a part of my fingerprint to one of them already. When in doubt, buy MAX232A chips from vendors that generally deal in genuine parts."
- note added: "This is considered a 5-wire hookup, for obvious reasons. Some computers require an active DCD to enable communication, it is therefore linked to DSR as a way around that."
- note removed: "C2-C5 must be electrolytic 1uF when using older or cheaper MAX232 variants, these can be replaced with standard 100nF when used with MAX232A."
- title: BulkyModem Module (RS-232) -> BulkyModem-32 Mini (RS-232)
Changed lines of the file:
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@@
 	(paper "A4")
 	(title_block
-		(title "BulkyModem Module (RS-232)")
+		(title "BulkyModem-32 Mini (RS-232)")
 		(rev "A")
 	)
@@
 		)
 	)
-	(text "C2-C5 must be electrolytic 1uF when using\nolder or cheaper MAX232 variants, these\ncan be replaced with standard 100nF\nwhen used with MAX232A."
+	(text "C2-C5 must be electrolytic 1uF when using\nolder or cheaper MAX232 variants, these\ncan be replaced with standard 100nF\nwhen used with the MAX232A."
 		(exclude_from_sim no)
 		(at 156.21 147.32 0)
@@
 		)
 	)
+	(text "This is considered a 5-wire hookup,\nfor obvious reasons. Some computers \nrequire an active DCD to enable\ncommunication, it is therefore linked\nto DSR as a way around that."
+		(exclude_from_sim no)
+		(at 124.46 38.1 0)
+		(effects
+			(font
+				(size 1.27 1.27)
+			)
+		)
+	)
+	(text "I know that there are 3.3v versions of these chips available, but as\nI regularly work with 5v - those are the chips that I have available.\nBesides, there are lots of bad cloned chips and I accidentally lost\na part of my fingerprint to one of them already. When in doubt, buy\nMAX232A chips from vendors that generally deal in genuine parts."
+		(exclude_from_sim no)
+		(at 241.3 93.98 0)
+		(effects
+			(font
+				(size 1.27 1.27)
+			)
+		)
+	)
