File: BulkyModem-32 Mini/BulkyModem-32 Mini.kicad_pcb (KiCad board)
At the start: 2 copper layers, 38.7 x 73 mm, 26 parts, among them J1 SD_CARD, J2 DCE, U3 MAX232, U6 74HCT32

Commit message: ESP32 Mini cleanup
Parts:
- A1: footprint esp32_dev_board:ESP32-WROOM-32D_30 -> esp32_dev_board:ESP32-WROOM-32D_30_Alternate

Commit message: Small build tweaks
Parts:
- R18, R5: value 10k* -> 10k
Other:
- board text added: "ESP32 Mini Module (rev. B)"
- board text removed: "ESP32 Mini Module (rev. A)"
Changed lines of the file:
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@@
 			)
 		)
-		(property "Value" "10k*"
+		(property "Value" "10k"
 			(at 3.81 0 270)
 			(layer "F.SilkS")
-			(hide yes)
 			(effects
 				(font
@@
 		(sheetname "Root")
 		(sheetfile "BulkyModem-32 Mini.kicad_sch")
-		(attr through_hole dnp)
+		(attr through_hole)
 		(fp_line
 			(start 8.35 -1.37)
@@
 		(tags "Diode DO-35_SOD27 series Axial Horizontal pin pitch 7.62mm  length 4mm diameter 2mm")
 		(property "Reference" "D14"
-			(at 3.81 0 90)
+			(at 4.445 0 90)
 			(layer "F.SilkS")
 			(effects
@@
 			)
 		)
-		(property "Value" "10k*"
+		(property "Value" "10k"
 			(at 3.937 0 270)
 			(layer "F.SilkS")
-			(hide yes)
 			(effects
 				(font
@@
 		(sheetname "Root")
 		(sheetfile "BulkyModem-32 Mini.kicad_sch")
-		(attr through_hole dnp)
+		(attr through_hole)
 		(fp_line
 			(start 8.35 -1.37)
@@
 		(tags "Diode DO-35_SOD27 series Axial Horizontal pin pitch 7.62mm  length 4mm diameter 2mm")
 		(property "Reference" "D15"
-			(at 3.81 0 90)
+			(at 4.445 0 90)
 			(layer "F.SilkS")
 			(effects
 				(font
-					(size 1 1)
-					(thickness 0.15)
+					(size 0.8 0.8)
+					(thickness 0.1)
 				)
 			)
@@
 		)
 	)
-	(gr_text "ESP32 Mini Module (rev. A)"
+	(gr_text "ESP32 Mini Module (rev. B)"
 		(at 108.458 59.944 0)
 		(layer "B.SilkS")
