File: BulkyModem-32 Mini/BulkyModem-32 Mini.kicad_sch (KiCad schematic)
At the start: 7 parts, among them J1 SD_CARD, U6 74HCT32

Commit message: ESP32 Mini cleanup
Parts:
- A1: footprint esp32_dev_board:ESP32-WROOM-32D_30 -> esp32_dev_board:ESP32-WROOM-32D_30_Alternate
Other:
- note added: "* Install R5/R18 if noise is encountered, otherwise leave unpopulated."
- note removed: "* Install R18 if noise is encountered, otherwise leave unpopulated."
- moved on the sheet: D15, R5
Changed lines of the file:
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@@
 		(title "BulkyModem-32 Mini")
 		(rev "A")
-		(comment 3 "before I actually knew what I was doing.")
+		(comment 2 "can probably tell - it's intended for use with RS-232.")
+		(comment 3 "before I knew what I was doing. This version is based around the ESP32, and as you")
 		(comment 4 "A smaller version of the BulkyModem-32, initially created as a way to test things out")
 	)
@@
 	)
 	(junction
-		(at 243.84 134.62)
+		(at 246.38 81.28)
 		(diameter 0)
 		(color 0 0 0 0)
 	)
 	(junction
-		(at 246.38 81.28)
+		(at 246.38 134.62)
 		(diameter 0)
 		(color 0 0 0 0)
@@
 	(wire
 		(pts
-			(xy 243.84 134.62) (xy 248.92 134.62)
-		)
-		(stroke
-			(width 0)
-			(type default)
-		)
-	)
-	(wire
-		(pts
 			(xy 166.37 91.44) (xy 171.45 91.44)
 		)
@@
 	(wire
 		(pts
+			(xy 259.08 134.62) (xy 261.62 134.62)
+		)
+		(stroke
+			(width 0)
+			(type default)
+		)
+	)
+	(wire
+		(pts
 			(xy 53.34 172.72) (xy 57.15 172.72)
 		)
@@
 	(wire
 		(pts
+			(xy 246.38 134.62) (xy 251.46 134.62)
+		)
+		(stroke
+			(width 0)
+			(type default)
+		)
+	)
+	(wire
+		(pts
 			(xy 224.79 68.58) (xy 228.6 68.58)
 		)
@@
 	(wire
 		(pts
-			(xy 243.84 133.35) (xy 243.84 134.62)
+			(xy 246.38 133.35) (xy 246.38 134.62)
 		)
 		(stroke
@@
 	(wire
 		(pts
-			(xy 243.84 134.62) (xy 114.3 134.62)
+			(xy 114.3 134.62) (xy 246.38 134.62)
 		)
 		(stroke
@@
 		)
 	)
-	(text "* Install R18 if noise is encountered,\notherwise leave unpopulated."
-		(exclude_from_sim no)
-		(at 236.22 88.9 0)
+	(text "* Install R5/R18 if noise is encountered,\notherwise leave unpopulated."
+		(exclude_from_sim no)
+		(at 238.76 105.41 0)
 		(effects
 			(font
@@
 	(global_label "ESP_CTS"
 		(shape input)
-		(at 256.54 134.62 0)
+		(at 261.62 134.62 0)
 		(effects
 			(font
@@
 		)
 		(property "Intersheetrefs" "${INTERSHEET_REFS}"
-			(at 256.54 134.62 0)
+			(at 261.62 134.62 0)
 			(effects
 				(font
@@
 			)
 		)
-		(property "Footprint" "esp32_dev_board:ESP32-WROOM-32D_30"
+		(property "Footprint" "esp32_dev_board:ESP32-WROOM-32D_30_Alternate"
 			(at 146.05 105.41 0)
 			(effects
@@
 	(symbol
 		(lib_id "Device:R")
-		(at 243.84 129.54 0)
+		(at 246.38 129.54 0)
 		(unit 1)
 		(exclude_from_sim no)
@@
 		(dnp yes)
 		(property "Reference" "R5"
-			(at 241.935 128.905 0)
+			(at 244.475 128.905 0)
 			(effects
 				(font
@@
 		)
 		(property "Value" "10k*"
-			(at 241.935 130.81 0)
+			(at 244.475 130.81 0)
 			(effects
 				(font
@@
 		)
 		(property "Footprint" "resistor:R_Axial_DIN0207_L6.3mm_D2.5mm_P10.16mm_Horizontal"
-			(at 242.062 129.54 90)
+			(at 244.602 129.54 90)
 			(effects
 				(font
@@
 		)
 		(property "Datasheet" "~"
-			(at 243.84 129.54 0)
+			(at 246.38 129.54 0)
 			(effects
 				(font
@@
 		)
 		(property "Description" "Resistor"
-			(at 243.84 129.54 0)
+			(at 246.38 129.54 0)
 			(effects
 				(font
@@
 	(symbol
 		(lib_id "power:+3.3V")
-		(at 243.84 125.73 0)
+		(at 246.38 125.73 0)
 		(unit 1)
 		(exclude_from_sim no)
@@
 		(dnp no)
 		(property "Reference" "#PWR01"
-			(at 243.84 129.54 0)
+			(at 246.38 129.54 0)
 			(effects
 				(font
@@
 		)
 		(property "Value" "+3.3V"
-			(at 244.221 121.3358 0)
+			(at 246.761 121.3358 0)
 			(effects
 				(font
@@
 		)
 		(property "Footprint" ""
-			(at 243.84 125.73 0)
+			(at 246.38 125.73 0)
 			(effects
 				(font
@@
 		)
 		(property "Datasheet" ""
-			(at 243.84 125.73 0)
+			(at 246.38 125.73 0)
 			(effects
 				(font
@@
 		)
 		(property "Description" "Power symbol creates a global label with name \"+3.3V\""
-			(at 243.84 125.73 0)
+			(at 246.38 125.73 0)
 			(effects
 				(font
@@
 	(symbol
 		(lib_id "Diode:1N4148")
-		(at 252.73 134.62 180)
+		(at 255.27 134.62 180)
 		(unit 1)
 		(exclude_from_sim no)
@@
 		(dnp no)
 		(property "Reference" "D15"
-			(at 252.73 129.1082 0)
+			(at 255.27 129.1082 0)
 			(effects
 				(font
@@
 		)
 		(property "Value" "1N4148"
-			(at 252.73 131.4196 0)
+			(at 255.27 131.4196 0)
 			(effects
 				(font
@@
 		)
 		(property "Footprint" "Diode_THT:D_DO-35_SOD27_P7.62mm_Horizontal"
-			(at 252.73 130.175 0)
+			(at 255.27 130.175 0)
 			(effects
 				(font
@@
 		)
 		(property "Datasheet" "https://assets.nexperia.com/documents/data-sheet/1N4148_1N4448.pdf"
-			(at 252.73 134.62 0)
+			(at 255.27 134.62 0)
 			(effects
 				(font
@@
 		)
 		(property "Description" "100V 0.15A standard switching diode, DO-35"
-			(at 252.73 134.62 0)
+			(at 255.27 134.62 0)
 			(effects
 				(font
@@
 		)
 		(property "Sim.Device" "D"
-			(at 252.73 134.62 0)
+			(at 255.27 134.62 0)
 			(effects
 				(font
@@
 		)
 		(property "Sim.Pins" "1=K 2=A"
-			(at 252.73 134.62 0)
-			(effects
-				(font
+			(at 255.27 134.62 0)
+			(effects
+				(font

Commit message: Small build tweaks
Parts:
- R18, R5: value 10k* -> 10k; now fitted
Other:
- note removed: "* Install R5/R18 if noise is encountered, otherwise leave unpopulated."
Changed lines of the file:
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@@
-		)
-	)
-	(text "* Install R5/R18 if noise is encountered,\notherwise leave unpopulated."
-		(exclude_from_sim no)
-		(at 238.76 105.41 0)
-		(effects
-			(font
-				(size 1.27 1.27)
-			)
-			(justify left bottom)
 		)
 	)
@@
 		(in_bom yes)
 		(on_board yes)
-		(dnp yes)
+		(dnp no)
 		(property "Reference" "R18"
 			(at 244.475 75.565 0)
@@
 			)
 		)
-		(property "Value" "10k*"
+		(property "Value" "10k"
 			(at 244.475 77.47 0)
 			(effects
@@
 		(in_bom yes)
 		(on_board yes)
-		(dnp yes)
+		(dnp no)
 		(property "Reference" "R5"
 			(at 244.475 128.905 0)
@@
 			)
 		)
-		(property "Value" "10k*"
+		(property "Value" "10k"
 			(at 244.475 130.81 0)
 			(effects

Commit message: Just clarification
Other:
- note added: "RI"
Changed lines of the file:
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@@
 	)
 	(no_connect
-		(at 125.73 71.12)
+		(at 120.65 71.12)
+	)
+	(wire
+		(pts
+			(xy 120.65 71.12) (xy 125.73 71.12)
+		)
+		(stroke
+			(width 0)
+			(type default)
+		)
 	)
 	(wire
@@
 	(text "SND"
 		(exclude_from_sim no)
-		(at 125.73 76.2 0)
+		(at 121.92 76.2 0)
 		(effects
 			(font
 				(size 1.27 1.27)
 			)
-			(justify right bottom)
-		)
-	)
-	(text "DSR"
+			(justify left bottom)
+		)
+	)
+	(text "RI"
 		(exclude_from_sim no)
-		(at 124.46 86.36 0)
+		(at 121.92 71.12 0)
 		(effects
 			(font
 				(size 1.27 1.27)
 			)
-			(justify right bottom)
+			(justify left bottom)
+		)
+	)
+	(text "DSR"
+		(exclude_from_sim no)
+		(at 121.92 86.36 0)
+		(effects
+			(font
+				(size 1.27 1.27)
+			)
+			(justify left bottom)
 		)
 	)
@@
 	(text "DTR"
 		(exclude_from_sim no)
-		(at 124.46 81.28 0)
+		(at 121.92 81.28 0)
 		(effects
 			(font
 				(size 1.27 1.27)
 			)
-			(justify right bottom)
-		)
-	)
+			(justify left bottom)
+		)
+	)
