File: BulkyModem Terminal/BulkyModem Terminal.kicad_sch (KiCad schematic)
At the start: 10 parts, among them M1 Mounting, M2 Mounting, M3 Mounting, M4 Mounting, U1 Pico

Commit message: Part of a layout
Parts:
- added SW1: RESET, Button_Switch_THT:SW_Tactile_SPST_Angled_PTS645Vx39-2LFS, symbol Switch:SW_Push
- added SW2: DEFAULTS, Button_Switch_THT:SW_Tactile_SPST_Angled_PTS645Vx39-2LFS, symbol Switch:SW_Push
Connections:
- net DEFAULTS: now also SW2.2
- net GND: now also SW1.1, SW2.1
- net RESET: now also SW1.2
Other:
- note added: "These switches are duplicated on the front panel. While no harm will come from installing both, you only need one set."

Commit message: Small build tweaks
Parts:
- D1, D3: value 1n4148 -> 1N4148
- R1, R2: value 1K -> 1k
Changed lines of the file:
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@@
 			)
 		)
-		(property "Value" "1n4148"
+		(property "Value" "1N4148"
 			(at 199.39 82.55 0)
 			(effects
@@
 			)
 		)
-		(property "Value" "1K"
+		(property "Value" "1k"
 			(at 184.15 73.66 0)
 			(effects
@@
 			)
 		)
-		(property "Value" "1K"
+		(property "Value" "1k"
 			(at 189.23 73.66 0)
 			(effects
@@
 			)
 		)
-		(property "Value" "1n4148"
+		(property "Value" "1N4148"
 			(at 199.39 92.71 0)
 			(effects
