File: BulkyModem Terminal/VGA.kicad_sch (KiCad schematic)
At the start: 10 parts, among them J4 VGA

Commit message: Fixed VGA footprint to match cheap parts
Parts:
- J4: footprint VGA_DSUB:DSUB-15-L77HDE15SD1CH4F -> VGA_DSUB:DSUB-15
Changed lines of the file:
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@@
 			)
 		)
-		(property "Footprint" "VGA_DSUB:DSUB-15-L77HDE15SD1CH4F"
+		(property "Footprint" "VGA_DSUB:DSUB-15"
 			(at 149.86 96.52 0)
 			(effects

Commit message: Small build tweaks
Parts:
- R11, R7: value 1K -> 1k
Changed lines of the file:
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@@
 			)
 		)
-		(property "Value" "1K"
+		(property "Value" "1k"
 			(at 181.61 98.6536 90)
 			(effects
@@
 			)
 		)
-		(property "Value" "1K"
+		(property "Value" "1k"
 			(at 181.61 70.7136 90)
 			(effects
