File: faceplates/BulkyModem Terminal FA1/BulkyModem Terminal FA1.kicad_pcb (KiCad board)
At the start: 2 copper layers, 100 x 100 mm, 10 parts, among them M1 Mounting, M2 Mounting, M3 Mounting, M4 Mounting

Commit message: Slightly move labels
Parts:
- moved REF** 0.38 mm to (153.3, 57.8)
Changed lines of the file:
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@@
 		(locked yes)
 		(layer "B.Cu")
-		(at 153.67 57.785 180)
+		(at 153.289 57.785 180)
 		(property "Reference" "REF**"
 			(at 0 1.016 180)
@@
 	)
 	(gr_text "VGA"
-		(at 153.461 55.245 0)
+		(at 153.289 55.245 0)
 		(layer "B.SilkS")
 		(effects
@@
 			(polygon
 				(pts
-					(xy 154.945263 56.245) (xy 154.945263 56.073053) (xy 155.126736 56.073053) (xy 155.126736 55.901106)
-					(xy 155.298683 55.901106) (xy 155.298683 55.025739) (xy 154.948683 55.025739) (xy 154.948683 55.901106)
-					(xy 154.595263 55.901106) (xy 154.595263 55.025739) (xy 154.251369 55.025739) (xy 154.251369 55.901106)
-					(xy 154.423316 55.901106) (xy 154.423316 56.073053) (xy 154.595263 56.073053) (xy 154.595263 56.245)
-				)
-			)
-			(polygon
-				(pts
-					(xy 153.901613 56.245) (xy 153.901613 56.073053) (xy 154.07356 56.073053) (xy 154.07356 55.197686)
-					(xy 153.901613 55.197686) (xy 153.901613 55.025739) (xy 153.198194 55.025739) (xy 153.198194 55.197686)
-					(xy 153.026247 55.197686) (xy 153.026247 55.372808) (xy 153.376247 55.372808) (xy 153.376247 55.200861)
-					(xy 153.72356 55.200861) (xy 153.72356 56.069877) (xy 153.376247 56.069877) (xy 153.376247 55.716702)
-					(xy 153.549904 55.716702) (xy 153.549904 55.54158) (xy 153.026247 55.54158) (xy 153.026247 56.073053)
-					(xy 153.198194 56.073053) (xy 153.198194 56.245)
-				)
-			)
-			(polygon
-				(pts
-					(xy 152.495019 55.197686) (xy 152.676491 55.197686) (xy 152.676491 55.369633) (xy 152.848438 55.369633)
-					(xy 152.848438 56.245) (xy 152.498438 56.245) (xy 152.498438 55.716702) (xy 152.145019 55.716702)
-					(xy 152.145019 56.245) (xy 151.801125 56.245) (xy 151.801125 55.54158) (xy 152.145019 55.54158)
-					(xy 152.498438 55.54158) (xy 152.498438 55.369633) (xy 152.145019 55.369633) (xy 152.145019 55.54158)
-					(xy 151.801125 55.54158) (xy 151.801125 55.369633) (xy 151.973072 55.369633) (xy 151.973072 55.197686)
-					(xy 152.145019 55.197686) (xy 152.145019 55.025739) (xy 152.495019 55.025739)
-				)
-			)
+					(xy 154.773263 56.245) (xy 154.773263 56.073053) (xy 154.954736 56.073053) (xy 154.954736 55.901106)
+					(xy 155.126683 55.901106) (xy 155.126683 55.025739) (xy 154.776683 55.025739) (xy 154.776683 55.901106)
+					(xy 154.423263 55.901106) (xy 154.423263 55.025739) (xy 154.079369 55.025739) (xy 154.079369 55.901106)
+					(xy 154.251316 55.901106) (xy 154.251316 56.073053) (xy 154.423263 56.073053) (xy 154.423263 56.245)
+				)
+			)
+			(polygon
+				(pts
+					(xy 153.729613 56.245) (xy 153.729613 56.073053) (xy 153.90156 56.073053) (xy 153.90156 55.197686)
+					(xy 153.729613 55.197686) (xy 153.729613 55.025739) (xy 153.026194 55.025739) (xy 153.026194 55.197686)
+					(xy 152.854247 55.197686) (xy 152.854247 55.372808) (xy 153.204247 55.372808) (xy 153.204247 55.200861)
+					(xy 153.55156 55.200861) (xy 153.55156 56.069877) (xy 153.204247 56.069877) (xy 153.204247 55.716702)
+					(xy 153.377904 55.716702) (xy 153.377904 55.54158) (xy 152.854247 55.54158) (xy 152.854247 56.073053)
+					(xy 153.026194 56.073053) (xy 153.026194 56.245)
+				)
+			)
+			(polygon
+				(pts
+					(xy 152.323019 55.197686) (xy 152.504491 55.197686) (xy 152.504491 55.369633) (xy 152.676438 55.369633)
+					(xy 152.676438 56.245) (xy 152.326438 56.245) (xy 152.326438 55.716702) (xy 151.973019 55.716702)
+					(xy 151.973019 56.245) (xy 151.629125 56.245) (xy 151.629125 55.54158) (xy 151.973019 55.54158)
+					(xy 152.326438 55.54158) (xy 152.326438 55.369633) (xy 151.973019 55.369633) (xy 151.973019 55.54158)
+					(xy 151.629125 55.54158) (xy 151.629125 55.369633) (xy 151.801072 55.369633) (xy 151.801072 55.197686)
+					(xy 151.973019 55.197686) (xy 151.973019 55.025739) (xy 152.323019 55.025739)
+				)
+			)
