File: BulkyModem Module Panel/BulkyModem Module Panel.kicad_pcb (KiCad board)
At the start: 2 copper layers, 100 x 23.2 mm, 20 parts, among them J1 Front Panel, M1 Mounting_Pin, M2 Mounting_Pin, M3 Mounting_Pin, M4 Mounting_Pin, SW1 MODE, SW2 POW

Commit message: Smaller build tweaks
Parts:
- removed D3, D4: 1N4148, Diode_THT:D_DO-35_SOD27_P7.62mm_Horizontal
- removed JP1: BYPASS, solder_bridge:bridge
- removed R1: 470, Resistor_THT:R_Axial_DIN0207_L6.3mm_D2.5mm_P10.16mm_Horizontal
Connections:
- net /LED_C64 renamed /LED.C64
- net /LED_CTS renamed /LED.CTS
- net /LED_DCD renamed /LED.DCD
- net /LED_POW renamed /LED.POW
- net /LED_RI renamed /LED.RI
- net /LED_RS232 renamed /LED.RS232
- net /LED_RTS renamed /LED.RTS
- net /LED_RX renamed /LED.RX
- net /LED_TX renamed /LED.TX
- D17 pad 2: Net-(D17-Pad2) -> VCC
- J1 pad 13: (no net) -> unconnected-(J1-N.C.-Pad13)
- J1 pad 14: (no net) -> unconnected-(J1-N.C.-Pad14)
- J1 pad 15: (no net) -> unconnected-(J1-N.C.-Pad15)
- J1 pad 16: (no net) -> unconnected-(J1-N.C.-Pad16)
- J1 pad 17: VSB -> unconnected-(J1-VSB-Pad17)
- J1 pad 4: (no net) -> unconnected-(J1-STB-Pad4)
- SW1 pad 1: (no net) -> unconnected-(SW1A-A-Pad1)
- SW1 pad 4: (no net) -> unconnected-(SW1B-A-Pad4)
- SW1 pad 5: (no net) -> unconnected-(SW1B-B-Pad5)
- SW1 pad 6: (no net) -> unconnected-(SW1B-C-Pad6)
- SW2 pad 1: (no net) -> unconnected-(SW2A-A-Pad1)
- SW2 pad 4: (no net) -> unconnected-(SW2B-A-Pad4)
Routing:
- net Net-(D17-Pad2): track 41.6 -> 0.00 mm
- net Net-(D4-Pad2): track 26.1 -> 0.00 mm
- net VSB: track 24.8 -> 0.00 mm, vias 2 -> 0
- net VCC: track 119.8 -> 116.2 mm
Other:
- net class Default removed
- net class PWR removed
- board text added: "BulkyModem Module Panel (rev. C) github.com/tebl"
- board text removed: "BulkyModem Module Panel (rev. B) github.com/tebl"
