File: BulkyModem-32 Module/BulkyModem-32 Module.kicad_pcb (KiCad board)
At the start: 2 copper layers, 100 x 100 mm, 68 parts, among them J1 DC IN, J2 DCE, J3 Module_Panel, J4 SD_CARD, J5 C64_Modem_OUT, K1 HK19F-DC, M1 Mounting, M2 Mounting, M3 Mounting, M4 Mounting, U1 74HCT244, U2 74HCT04, U3 MAX232, U4 MAX232, U6 74HCT32

Commit message: Smaller build tweaks
Parts:
- added SW1: FACTORY, Button_Switch_THT:SW_Tactile_SPST_Angled_PTS645Vx39-2LFS, F.Cu at (167.3, 125.0)
- D1: value 1n4148 -> 1N4148
- moved C1 0.64 mm to (84.5, 73.7)
Connections:
- A1 pad 2: unconnected-(A1-VP-Pad2) -> Net-(A1-VP)
Routing:
- net Net-(A1-VP): track 0.00 -> 66.5 mm, vias 0 -> 2
- net +5V: track 560.4 -> 554.7 mm
- net AUDIO_TX: track 41.0 -> 36.6 mm
- net AUDIO_RX: track 46.5 -> 42.4 mm
- net VIN: track 64.8 -> 65.4 mm
Other:
- board text added: "ESP32 Module (rev. B) github.com/tebl"
- board text removed: "ESP32 Module (rev. A) github.com/tebl"
