File: BulkyModem-32 Module/power.kicad_sch (KiCad schematic)
At the start: 17 parts, among them J1 DC IN, K1 HK19F-DC, U2 74HCT04, U6 74HCT32

Commit message: Smaller build tweaks
Parts:
- D1: value 1n4148 -> 1N4148
Changed lines of the file:
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@@
 			)
 		)
-		(property "Value" "1n4148"
+		(property "Value" "1N4148"
 			(at 166.37 93.98 90)
 			(effects
@@
 			)
 		)
-		(property "Datasheet" "~"
+		(property "Datasheet" "https://assets.nexperia.com/documents/data-sheet/1N4148_1N4448.pdf"
 			(at 175.26 93.98 0)
 			(effects
